File: hardware/01_Power_Input_USB.kicad_sch (KiCad schematic)
At the start: 43 parts, among them J1 1053131302 / 12V INPUT, J5 USB4105-GF-A-120, Q1 IPG20N06S4L-26, U1 LM74720QDRRRQ1, U2 TUSB321AIRWBR, U3 TPS259470LRPWR, U4 LMR43620MSC3RPERQ1

Commit message: Rebuild phase 2 schematic by function
Parts:
- added D17: BZT52H-C18-QX, Diode_SMD:D_SOD-123F, symbol LandyHeater:BZT52H_C18_QX_1K_2A
- added Q8: 2N7002KQ-13 USB CURRENT ISOLATOR, Package_TO_SOT_SMD:SOT-23, symbol LandyHeater:2N7002KQ_13_USB_CURRENT_ISOLATOR_1G_2S_3D
- added R72: 1M, Resistor_SMD:R_0603_1608Metric_Pad0.98x0.95mm_HandSolder, symbol LandyHeater:1M_11_22
- added R73: 100k, Resistor_SMD:R_0603_1608Metric_Pad0.98x0.95mm_HandSolder, symbol LandyHeater:100k_11_22
- added R74: 100R, Resistor_SMD:R_0603_1608Metric_Pad0.98x0.95mm_HandSolder, symbol LandyHeater:100R_11_22
- C11: value 4.7uF 50V -> 4.7uF 50V X7R 10%; footprint Capacitor_SMD:C_0805_2012Metric_Pad1.18x1.45mm_HandSolder -> Capacitor_SMD:C_1210_3225Metric_Pad1.33x2.70mm_HandSolder; symbol LandyHeater:4_7uF_50V_11_22 -> LandyHeater:4_7uF_50V_X7R_10__11_22; MPN (none) -> GCJ32ER71H475KA12; Manufacturer (none) -> Murata; Notes (none) -> LMR43620 local input capacitor; DC-bias effective capacitan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
- C13, C14: value 22uF 10V -> 22uF 10V X7R 10%; footprint Capacitor_SMD:C_0805_2012Metric_Pad1.18x1.45mm_HandSolder -> Capacitor_SMD:C_1206_3216Metric_Pad1.33x1.80mm_HandSolder; symbol LandyHeater:22uF_10V_11_22 -> LandyHeater:22uF_10V_X7R_10__11_22; MPN (none) -> GCJ31CR71A226KE01; Manufacturer (none) -> Murata; Notes (none) -> Effective capacitance at 3.3V/temperature must be verified
- C4: Notes PD slew; validate inrush -> PD slew to GND per LM74720-Q1 Figure 9-1; validate inrush/S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
- J1: symbol LandyHeater:1053131302_12V_INPUT_11_22 -> LandyHeater:1053131302_12V_INPUT_1BATT_12V_IN_2GND
- L1: Notes (none) -> PROVISIONAL generic footprint; verify against Coilcraft lan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
- L2: value 3.3uH 3A -> 2.2uH 5.6A Isat; symbol LandyHeater:3_3uH_3A_11_22 -> LandyHeater:2_2uH_5_6A_Isat_11_22; MPN XAL4020-332MEB -> XAL4020-222MEC; Notes (none) -> TI Table 8-2 fixed 3.3V/2.2MHz; 20% tolerance
- R3: Notes (none) -> TI Figure 9-1 R5
- R5: Notes (none) -> TUSB321 OUT1 pull-up; referenced only to TUSB321 VDD
- R6: Notes (none) -> TUSB321 OUT2 pull-up; test point is 5-V domain
- U1: footprint Package_SON:WSON-12-1EP_3x3mm_P0.5mm_EP1.5x2.5mm_ThermalVias -> Package_SON:WSON-12-1EP_3x3mm_P0.5mm_EP1.5x2.5mm
- U3: Notes (none) -> PROVISIONAL generic RPW footprint; verify/replace from offi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
- U4: Notes (none) -> PROVISIONAL project-local RPE footprint; verify/replace fro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
Connections:
- net 3V3_CORE: now also R73.1; no longer R5.1, R6.1
- net GND: now also C4.2, Q8.2 (S), R72.2
- net Q2_GATE_FET: now also D17.1 (K), R74.1; no longer C4.1
- net USB_VBUS: now also R5.1, R6.1
- net VIN_12V_PROTECTED: now also D17.2 (A); no longer C4.2
- net BATT_12V renamed BATT_12V_IN
- net Q1_GATE: no longer names the net of Q1.2 (G1), U1.1 (GATE)
- net USB_HIGH_CURRENT_N renamed USB_CURRENT_OUT1
- net USB_CURRENT_OUT1: now also Q8.1 (G), R72.1
- new net: C4.1, R74.2
- new net USB_HIGH_CURRENT: Q8.3 (D), R73.2
Other:
- note added: "12-V INPUT / REVERSE BATTERY / OV CUTOFF"
- note added: "FLOW: J1 -> TVS + LM74720/Q1 -> FILTER -> VIN_SYS"
- note added: "FLOW: J5 -> TUSB321 + TPS259470 -> POWER OR -> LMR43620/L2 -> 3V3_CORE"
- note added: "RTN exposed pad of U1 MUST FLOAT"
- note added: "USB-C UFP / CURRENT DETECTION / TRUE REVERSE BLOCKING"
- moved on the sheet: C1, C10, C11, C12, C13, C14, C2, C3, C4, C5, C6, C7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

Commit message: Redraw phase 2 schematic with visible functional wiring
Parts:
- C1, C2: Circuit label (none) -> 1uF 50V X7R
- C10: Circuit label (none) -> 1uF 10V
- C11: Circuit label (none) -> GCJ32ER71H475KA12
- C12: Circuit label (none) -> 100nF 50V
- C13, C14: Circuit label (none) -> GCJ31CR71A226KE01
- C3: Circuit label (none) -> 100nF 50V X7R
- C4: Circuit label (none) -> 10nF 50V
- C5: Circuit label (none) -> 4.7uF 50V X7R
- C6: Circuit label (none) -> 22uF 25V X7R
- C7: Circuit label (none) -> 100nF
- C8: Circuit label (none) -> 10nF
- C9: Circuit label (none) -> 100nF 10V
- D1: Circuit label (none) -> TPSMB18CA-VR
- D17: Circuit label (none) -> BZT52H-C18-QX
- D2: Circuit label (none) -> ESD5Z5.0T1G
- FB1: Circuit label (none) -> MPZ2012S221A
- J1: Circuit label (none) -> 12 V INPUT
- J5: Circuit label (none) -> USB-C
- L1: Circuit label (none) -> XPL2010-104ML
- L2: Circuit label (none) -> XAL4020-222MEC
- NT1: Circuit label (none) -> POWER OR
- Q1: Circuit label (none) -> IPG20N06S4L-26
- Q8: Circuit label (none) -> 2N7002KQ-13
- R1, R7: Circuit label (none) -> 100k 1%
- R10, R73: Circuit label (none) -> 100k
- R2: Circuit label (none) -> 7.15k 1%
- R3, R68: Circuit label (none) -> 0R
- R4: Circuit label (none) -> 900k 1%
- R5, R6: Circuit label (none) -> 220k
- R72: Circuit label (none) -> 1M
- R74: Circuit label (none) -> 100R
- R8: Circuit label (none) -> 26.1k 1%
- R9: Circuit label (none) -> 3.32k 1%
- U1: Circuit label (none) -> LM74720QDRRRQ1
- U2: Circuit label (none) -> TUSB321AIRWBR
- U3: Circuit label (none) -> TPS259470LRPWR
- U4: Circuit label (none) -> LMR43620MSC3RPERQ1
Connections:
- net BOOST_CAP: no longer names the net of C1.1, U1.10 (CAP)
- net BOOST_LX: no longer names the net of L1.2, U1.9 (LX)
- net BUCK_BOOT: no longer names the net of C9.1, U4.6 (BOOT)
- net BUCK_PGOOD: no longer names the net of R10.2, U4.2 (PGOOD)
- net BUCK_SW: no longer names the net of C9.2, L2.1, U4.5 (SW)
- net BUCK_VCC: no longer names the net of C10.1, U4.7 (VCC)
- net CC1: no longer names the net of J5.A5 (CC1), U2.1 (CC1)
- net CC2: no longer names the net of J5.B5 (CC2), U2.2 (CC2)
- net FET_COMMON: no longer names the net of C1.2, C2.1, L1.1, Q1.5 (D2), Q1.6 (D2), Q1.7 (D1), Q1.8 (D1), U1.11 (VS), U1.12 (C)
- net OV_SENSE: no longer names the net of R1.2, R2.1, U1.5 (OV)
- net OV_TOP: no longer names the net of R1.1, U1.4 (SW)
- net Q2_GATE: no longer names the net of R3.1, U1.8 (PD)
- net Q2_GATE_FET: no longer names the net of D17.1 (K), Q1.4 (G2), R3.2, R74.1
- net USB_CURRENT_OUT1: no longer names the net of Q8.1 (G), R5.2, R72.1, U2.7 (OUT1)
- net USB_DVDT: no longer names the net of C8.1, U3.7 (DVDT)
- net USB_ILM: no longer names the net of R9.1, U3.9 (ILM)
- net USB_OVLO: no longer names the net of R7.2, R8.1, U3.2 (OVLO)
- net USB_SHIELD: no longer names the net of J5.SH (SHIELD), R68.1
- net USB_VBUS_DET: no longer names the net of R4.2, U2.5 (VBUS_DET)
Other:
- note added: "12 V INPUT - TVS - IDEAL DIODE - FILTER"
- note added: "POWER MERGE TO VIN_SYS"
- note added: "RTN/EP OF U1 MUST FLOAT"
- note added: "TRUE REVERSE BLOCKING - 1 A USB LIMIT"
- note added: "USB-C SINK - CC DETECTION - eFUSE - POWER OR"
- note added: "VIN_SYS - AUTOMOTIVE BUCK - 3V3_CORE"
- note removed: "12-V INPUT / REVERSE BATTERY / OV CUTOFF"
- note removed: "FLOW: J1 -> TVS + LM74720/Q1 -> FILTER -> VIN_SYS"
- note removed: "FLOW: J5 -> TUSB321 + TPS259470 -> POWER OR -> LMR43620/L2 -> 3V3_CORE"
- note removed: "RTN exposed pad of U1 MUST FLOAT"
- note removed: "USB-C UFP / CURRENT DETECTION / TRUE REVERSE BLOCKING"
- moved on the sheet: C1, C10, C11, C12, C13, C14, C2, C3, C4, C5, C6, C7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
