File: hardware/02_ESP32_USB_Reset.kicad_sch (KiCad schematic)
At the start: 26 parts, among them SW1 RESET KMR221GLFS, SW2 BOOT KMR221GLFS, U5 ESP32-S3-WROOM-1U-N16R8, U6 TPS3808G33QDBVRQ1, U7 TPD2EUSB30DRTR

Commit message: Rebuild phase 2 schematic by function
Parts:
- added C40, C41, C42, C43, C44, C45, C46: 10pF C0G DNP, Capacitor_SMD:C_0603_1608Metric_Pad1.08x0.95mm_HandSolder, symbol LandyHeater:10pF_C0G_DNP_11_22
- added TP23: CHIP_PU, TestPoint:TestPoint_Pad_D1.0mm, symbol LandyHeater:CHIP_PU_11
- added TP24: BOOT_N, TestPoint:TestPoint_Pad_D1.0mm, symbol LandyHeater:BOOT_N_11
- C15: value 10uF 10V -> 22uF 10V X7R 10%; footprint Capacitor_SMD:C_0805_2012Metric_Pad1.18x1.45mm_HandSolder -> Capacitor_SMD:C_1206_3216Metric_Pad1.33x1.80mm_HandSolder; symbol LandyHeater:10uF_10V_11_22 -> LandyHeater:22uF_10V_X7R_10__11_22; MPN (none) -> GCJ31CR71A226KE01; Manufacturer (none) -> Murata; Notes (none) -> ESP32 local bulk; effective capacitance must be verified
- C16: value 1uF 10V -> 22uF 10V X7R 10%; footprint Capacitor_SMD:C_0603_1608Metric_Pad1.08x0.95mm_HandSolder -> Capacitor_SMD:C_1206_3216Metric_Pad1.33x1.80mm_HandSolder; symbol LandyHeater:1uF_10V_11_22 -> LandyHeater:22uF_10V_X7R_10__11_22; MPN (none) -> GCJ31CR71A226KE01; Manufacturer (none) -> Murata; Notes (none) -> ESP32 local bulk; effective capacitance must be verified
- U6: Notes (none) -> CT intentionally open for fixed nominal 20-ms reset delay
Connections:
- net BOOT_N: now also TP24.1
- net CHIP_PU: now also TP23.1
- net EPD_CS_N: now also C44.1
- net EPD_DC: now also C45.1
- net EPD_RESET_N: now also C46.1
- net EPD_SCLK: now also C42.1
- net EPD_SDIO_MOSI: now also C43.1
- net GND: now also C40.2, C41.2, C42.2, C43.2, C44.2, C45.2, C46.2
- net USB_D_N_ESP: now also C40.1
- net USB_D_P_ESP: now also C41.1
- net 1WIRE_DQ renamed 1WIRE_DQ_GPIO
- net U0TXD_TEST: no longer names the net of R16.2, TP6.1
- net USB_HIGH_CURRENT_N renamed USB_HIGH_CURRENT
Other:
- note added: "CT open = 20 ms reset delay (TPS3808)"
- note added: "ESP32-S3-WROOM-1U-N16R8 / SAFE RESET AND BOOT"
- note added: "FLOW: 3V3 -> TPS3808/RESET -> CHIP_PU | USB J5 -> ESD -> R14/R15 -> GPIO19/20 | GPIO -> SPI SERIES PARTS"
- note added: "USB tuning capacitors and SPI tuning capacitors: DNP"
- moved on the sheet: C15, C16, C17, C18, C19, R11, R12, R13, R14, R15, R16, R54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

Commit message: Redraw phase 2 schematic with visible functional wiring
Parts:
- C15, C16: Circuit label (none) -> GCJ31CR71A226KE01
- C17, C19: Circuit label (none) -> 100nF
- C18: Circuit label (none) -> 1uF
- C40, C41, C42, C43, C44, C45, C46: Circuit label (none) -> 10pF C0G DNP [DNP]
- R11, R12, R13: Circuit label (none) -> 10k
- R14, R15: Circuit label (none) -> 22R
- R16: Circuit label (none) -> 499R
- R54, R55, R56, R57, R58, R59: Circuit label (none) -> 33R
- SW1, SW2: Circuit label (none) -> KMR221GLFS
- U5: Circuit label (none) -> ESP32-S3-WROOM-1U-N16R8
- U6: Circuit label (none) -> TPS3808G33QDBVRQ1
- U7: Circuit label (none) -> TPD2EUSB30DRTR
Connections:
- net BOOT_N: no longer names the net of R13.2, SW2.1 (A), TP24.1, U5.27 (IO0)
- net CHIP_PU: no longer names the net of C18.1, R11.2, TP23.1, U5.3 (EN), U6.1 (RESET_N)
- net EPD_BUSY_GPIO: no longer names the net of R59.2, U5.12 (IO8)
- net EPD_CS_GPIO_N: no longer names the net of R56.1, U5.19 (IO11)
- net EPD_DC_GPIO: no longer names the net of R57.1, U5.20 (IO12)
- net EPD_RESET_GPIO_N: no longer names the net of R58.1, U5.21 (IO13)
- net EPD_SCLK_GPIO: no longer names the net of R54.1, U5.17 (IO9)
- net EPD_SDIO_GPIO: no longer names the net of R55.1, U5.18 (IO10)
- net RESET_MR_N: no longer names the net of R12.2, SW1.1 (A), U6.3 (MR_N)
- net U0RXD_TEST: no longer names the net of TP7.1, U5.36 (U0RXD/IO44)
- net U0TXD_RAW: no longer names the net of R16.1, U5.37 (U0TXD/IO43)
- net USB_D_N_ESP: no longer names the net of C40.1, R14.2, U5.13 (IO19/USB_D-)
- net USB_D_N_PROT: no longer names the net of R14.1, U7.5 (D1_OUT)
- net USB_D_P_ESP: no longer names the net of C41.1, R15.2, U5.14 (IO20/USB_D+)
- net USB_D_P_PROT: no longer names the net of R15.1, U7.4 (D2_OUT)
Other:
- note added: "CT OPEN = FIXED 20 ms RESET DELAY"
- note added: "E-PAPER SIGNAL CONDITIONING"
- note added: "ESP32-S3 MODULE"
- note added: "NATIVE USB PROTECTION"
- note added: "PROGRAMMING / STATUS TEST POINTS"
- note added: "RESET / BOOT / SUPERVISOR"
- note added: "USB AND SPI SHUNT CAPACITORS ARE DNP"
- note removed: "CT open = 20 ms reset delay (TPS3808)"
- note removed: "ESP32-S3-WROOM-1U-N16R8 / SAFE RESET AND BOOT"
- note removed: "FLOW: 3V3 -> TPS3808/RESET -> CHIP_PU | USB J5 -> ESD -> R14/R15 -> GPIO19/20 | GPIO -> SPI SERIES PARTS"
- note removed: "USB tuning capacitors and SPI tuning capacitors: DNP"
- moved on the sheet: C15, C16, C17, C18, C19, C40, C41, C42, C43, C44, C45, C46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
