File: hardware/03_Display_EPaper.kicad_sch (KiCad schematic)
At the start: 38 parts, among them J6 FH12-24S-0.5SH(55) E-PAPER, Q2 2N7002KQ-13, Q3 SI1308EDL-T1-GE3, U10 SN74AXC1T45DCKR, U8 TPS22919QDCKRQ1, U9 SN74AXC8T245PWR

Commit message: Rebuild phase 2 schematic by function
Parts:
- added C47, C48, C49, C50, C53: 100nF, Capacitor_SMD:C_0603_1608Metric_Pad1.08x0.95mm_HandSolder, symbol LandyHeater:100nF_11_22
- added TP34: DISPLAY_EN, TestPoint:TestPoint_Pad_D1.0mm, symbol LandyHeater:DISPLAY_EN_11
- C37: Notes (none) -> Good Display C11; VGL/PREVGL to GND
- L3: value 47uH 500mA -> 47uH 570mA; footprint Inductor_SMD:L_Changjiang_FNR3015S -> LandyHeater:PROVISIONAL_Murata_LQH3NPZ_JR; symbol LandyHeater:47uH_500mA_11_22 -> LandyHeater:47uH_570mA_11_22; MPN (none) -> LQH3NPZ470MJR; Manufacturer (none) -> Murata; Notes Good Display chapter 12; NR3015 class -> Good Display chapter 12; footprint is provisional pending o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
Connections:
- net 3V3_CORE: now also C47.1, C49.1
- net 3V3_DISPLAY_SW: now also C48.1, C50.1, C53.1
- net DISPLAY_EN: now also TP34.1
- net EPD_PREVGL: now also C37.1; no longer C37.2
- net EPD_VSL: no longer C37.1
- net GND: now also C37.2, U9.10 (A8), U9.8 (A6), U9.9 (A7), C47.2, C48.2, C49.2, C50.2, C53.2
- no-connect marks 12 -> 9
Other:
- note added: "DISPLAY POWER-OFF ISOLATION"
- note added: "FLOW: GPIO SPI -> AXC LEVEL/POWER-OFF ISOLATION -> J6 | 3V3_DISPLAY_SW -> BOOSTER -> PANEL RAILS"
- note added: "FPC contact side / pin-1 orientation: NOT VERIFIED until original sample inspection"
- note added: "GOOD DISPLAY CHAPTER 12 BOOSTER — DO NOT SUBSTITUTE TOPOLOGY"
- moved on the sheet: C20, C21, C22, C23, C24, C25, C26, C27, C36, C37, C38, D3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

Commit message: Redraw phase 2 schematic with visible functional wiring
Parts:
- C20: Circuit label (none) -> 1uF
- C21, C26: Circuit label (none) -> 4.7uF 25V
- C22, C23, C24, C25, C27, C36, C37, C38: Circuit label (none) -> 1uF 25V
- C47, C48, C49, C50, C53: Circuit label (none) -> 100nF
- D3, D4, D5: Circuit label (none) -> MBR0530T1G
- J6: Circuit label (none) -> E-PAPER FPC
- L3: Circuit label (none) -> LQH3NPZ470MJR
- Q2: Circuit label (none) -> 2N7002KQ-13
- Q3: Circuit label (none) -> SI1308EDL-T1-GE3
- R17, R18, R19, R60, R61, R62, R63, R64: Circuit label (none) -> 100k
- R20: Circuit label (none) -> 1M 1%
- R21: Circuit label (none) -> 2.2R 1%
- U10: Circuit label (none) -> SN74AXC1T45DCKR
- U8: Circuit label (none) -> TPS22919QDCKRQ1
- U9: Circuit label (none) -> SN74AXC8T245PWR
Connections:
- net EPD_BOOST_SW: no longer names the net of C26.1, D3.2 (A), L3.2, Q3.3 (D)
- net EPD_BUSY_PANEL: no longer names the net of J6.9, TP19.1, U10.4 (B)
- net EPD_CS_PANEL_N: no longer names the net of J6.12, R62.2, TP16.1, U9.19 (B3)
- net EPD_DC_PANEL: no longer names the net of J6.11, R63.1, TP17.1, U9.18 (B4)
- net EPD_GDR: no longer names the net of J6.2, Q3.1 (G), R20.1
- net EPD_LEVEL_OE_N: no longer names the net of Q2.3 (D), R18.2, U9.22 (OE_N)
- net EPD_NEG_PUMP: no longer names the net of C26.2, D4.1 (K), D5.2 (A)
- net EPD_PREVGH: no longer names the net of C27.1, C36.1, D3.1 (K), J6.21
- net EPD_PREVGL: no longer names the net of C37.1, D4.2 (A), J6.23
- net EPD_RESE: no longer names the net of J6.3, Q3.2 (S), R21.1
- net EPD_RESET_PANEL_N: no longer names the net of J6.10, R64.1, TP18.1, U9.17 (B5)
- net EPD_SCLK_PANEL: no longer names the net of J6.13, R60.1, TP14.1, U9.21 (B1)
- net EPD_SDIO_PANEL: no longer names the net of J6.14, R61.1, TP15.1, U9.20 (B2)
- net EPD_VCOM: no longer names the net of C38.1, J6.24
- net EPD_VDD: no longer names the net of C24.1, J6.18
- net EPD_VSH1: no longer names the net of C25.1, J6.20
- net EPD_VSH2: no longer names the net of C22.1, J6.5
- net EPD_VSL: no longer names the net of C36.2, J6.22
Other:
- note added: "DISPLAY LOAD SWITCH"
- note added: "FPC CONTACT SIDE / PIN 1: VERIFY ON PHYSICAL SAMPLE"
- note added: "GOOD DISPLAY CHAPTER 12 REFERENCE BOOSTER - DO NOT SUBSTITUTE TOPOLOGY"
- note added: "J6 FPC"
- note added: "POWER-OFF SIGNAL ISOLATION"
- note added: "REFERENCE BOOSTER / PANEL RAILS"
- note removed: "DISPLAY POWER-OFF ISOLATION"
- note removed: "FLOW: GPIO SPI -> AXC LEVEL/POWER-OFF ISOLATION -> J6 | 3V3_DISPLAY_SW -> BOOSTER -> PANEL RAILS"
- note removed: "FPC contact side / pin-1 orientation: NOT VERIFIED until original sample inspection"
- note removed: "GOOD DISPLAY CHAPTER 12 BOOSTER — DO NOT SUBSTITUTE TOPOLOGY"
- moved on the sheet: C20, C21, C22, C23, C24, C25, C26, C27, C36, C37, C38, C47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
