File: hardware/05_AUTOTERM_1Wire.kicad_sch (KiCad schematic)
At the start: 19 parts, among them J2 1053131304 / AUTOTERM, J3 1053131303 / 1-WIRE, U15 TPS22945DCKR, U16 TXU0202QDCURQ1, U17 TPS22945DCKR

Commit message: Rebuild phase 2 schematic by function
Parts:
- added C51: 100nF, Capacitor_SMD:C_0603_1608Metric_Pad1.08x0.95mm_HandSolder, symbol LandyHeater:100nF_11_22
- added TP25: AUTOTERM_TX_3V3, TestPoint:TestPoint_Pad_D1.0mm, symbol LandyHeater:AUTOTERM_TX_3V3_11
- added TP26: AUTOTERM_RX_3V3, TestPoint:TestPoint_Pad_D1.0mm, symbol LandyHeater:AUTOTERM_RX_3V3_11
- added TP27: CTRL_TX_TO_HEATER, TestPoint:TestPoint_Pad_D1.0mm, symbol LandyHeater:CTRL_TX_TO_HEATER_11
- added TP28: CTRL_RX_FROM_HEATER, TestPoint:TestPoint_Pad_D1.0mm, symbol LandyHeater:CTRL_RX_FROM_HEATER_11
- added TP29: 3V3_SENSOR_SW, TestPoint:TestPoint_Pad_D1.0mm, symbol LandyHeater:3V3_SENSOR_SW_11
- D7: symbol LandyHeater:PESD5V2S2UT_Q_1IO1_2GND_3IO2 -> LandyHeater:PESD5V2S2UT_Q_1K1_2K2_3A; Notes (none) -> Pins 1/2 cathodes to signals; pin 3 common anode to GND
- D8: symbol LandyHeater:PESD3V3S2UT_Q_1IO1_2GND_3IO2 -> LandyHeater:PESD3V3S2UT_Q_1K1_2K2_3A; Notes (none) -> Pins 1/2 cathodes to protected lines; pin 3 common anode to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
- J2: symbol LandyHeater:1053131304_AUTOTERM_11_22_33_44 -> LandyHeater:1053131304_AUTOTERM_1AUTOTERM_5V_2GND_3CTRL_TX_TO_HEATER_4CTRL_RX_FROM_HEATER
- J3: symbol LandyHeater:1053131303_1_WIRE_11_22_33 -> LandyHeater:1053131303_1_WIRE_13V3_SENSOR_SW_21WIRE_DQ_3GND
- R37: value 100R -> 0R; symbol LandyHeater:100R_11_22 -> LandyHeater:0R_11_22; Notes (none) -> Required populated 0-ohm tuning link
- TP11: value AUTOTERM_5V -> AUTOTERM_5V_PROTECTED; symbol LandyHeater:AUTOTERM_5V_11 -> LandyHeater:AUTOTERM_5V_PROTECTED_11
- U15: Notes 100mA-class protected heater supply; OC_N intentionally unu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 -> 100-mA current-limited protection; heater-side supply only
Connections:
- net 1WIRE_WIRE is gone; now on net 1WIRE_DQ: D8.1 (K1), J3.2 (1WIRE_DQ), R37.2
- net AUTOTERM_5V_IN is gone; now on net AUTOTERM_5V: C31.1, J2.1 (AUTOTERM_5V), U15.4 (ON), U15.5 (VIN)
- net 1WIRE_DQ: no longer R37.1
- net 3V3_CORE: now also C51.1
- net 3V3_SENSOR_SW: now also D8.2 (K2), TP29.1; no longer D8.3 (IO2)
- net AUTOTERM_5V: no longer C32.1, TP11.1, U15.1 (VOUT), U16.7 (VCCB)
- net AUTOTERM_RX_3V3: now also TP26.1
- net AUTOTERM_TX_3V3: now also TP25.1
- net GND: now also D7.3 (A), D8.3 (A), J2.2 (GND), C51.2; no longer D7.2 (GND), D8.2 (GND), J2.4
- removed net AUTOTERM_RX_WIRE: D7.3 (IO2), J2.3, R34.1
- net AUTOTERM_TX_WIRE renamed CTRL_TX_TO_HEATER
- net CTRL_TX_TO_HEATER: now also J2.3 (CTRL_TX_TO_HEATER), TP27.1; no longer J2.2
- new net 1WIRE_DQ_GPIO: R37.1
- new net AUTOTERM_5V_PROTECTED: C32.1, TP11.1, U15.1 (VOUT), U16.7 (VCCB)
- new net CTRL_RX_FROM_HEATER: D7.2 (K2), J2.4 (CTRL_RX_FROM_HEATER), R34.1, TP28.1
Other:
- note added: "1-WIRE — THREE DS18B20 / 2–5 m combined harness"
- note added: "AUTOTERM UART — 5-V side powered only by heater"
- note added: "FLOW: 3V3 -> TPS22945 -> SENSOR SUPPLY | GPIO4 -> 0R + ESD -> J3"
- note added: "FLOW: ESP32 UART -> TXU0202 -> SERIES + ESD -> J2"
- note added: "J2 PIN ORDER: 1=5V, 2=GND, 3=TX TO HEATER, 4=RX FROM HEATER"
- moved on the sheet: C31, C32, C33, C34, D7, D8, J2, J3, R32, R33, R34, R35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

Commit message: Redraw phase 2 schematic with visible functional wiring
Parts:
- C31, C33: Circuit label (none) -> 1uF
- C32, C34, C51: Circuit label (none) -> 100nF
- D7: Circuit label (none) -> PESD5V2S2UT-Q
- D8: Circuit label (none) -> PESD3V3S2UT-Q
- J2: Circuit label (none) -> AUTOTERM
- J3: Circuit label (none) -> 1-WIRE
- R32, R35: Circuit label (none) -> 100k
- R33, R34: Circuit label (none) -> 100R
- R36: Circuit label (none) -> 4.7k
- R37: Circuit label (none) -> 0R
- U15, U17: Circuit label (none) -> TPS22945DCKR
- U16: Circuit label (none) -> TXU0202QDCURQ1
Connections:
- net 1WIRE_DQ: no longer names the net of D8.1 (K1), J3.2 (1WIRE_DQ), R36.2, R37.2, TP12.1
- net AUTOTERM_RX_PROT: no longer names the net of R34.2, U16.1 (B2)
- net AUTOTERM_TX_PROT: no longer names the net of R33.1, U16.8 (B1Y)
- net CTRL_RX_FROM_HEATER: no longer names the net of D7.2 (K2), J2.4 (CTRL_RX_FROM_HEATER), R34.1, TP28.1
- net CTRL_TX_TO_HEATER: no longer names the net of D7.1 (K1), J2.3 (CTRL_TX_TO_HEATER), R33.2, TP27.1
Other:
- note added: "1-WIRE: LOAD SWITCH / PULL-UP -> SERIES / ESD -> J3"
- note added: "AUTOTERM UART: ESP32 -> LEVEL SHIFT -> SERIES -> ESD -> J2"
- note added: "J2: 1=5V, 2=GND, 3=TX TO HEATER, 4=RX FROM HEATER"
- note added: "THREE DS18B20 ON ONE 2-5 m COMBINED HARNESS"
- note removed: "1-WIRE — THREE DS18B20 / 2–5 m combined harness"
- note removed: "AUTOTERM UART — 5-V side powered only by heater"
- note removed: "FLOW: 3V3 -> TPS22945 -> SENSOR SUPPLY | GPIO4 -> 0R + ESD -> J3"
- note removed: "FLOW: ESP32 UART -> TXU0202 -> SERIES + ESD -> J2"
- note removed: "J2 PIN ORDER: 1=5V, 2=GND, 3=TX TO HEATER, 4=RX FROM HEATER"
- moved on the sheet: C31, C32, C33, C34, C51, D7, D8, J2, J3, R32, R33, R34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
