File: hardware/06_Controls_Diagnostics.kicad_sch (KiCad schematic)
At the start: 48 parts, among them J4 1053131305 / BUTTON+LED, J8 FH12-6S-0.5SH(55) FRONTLIGHT, Q4 2N7002KQ-13, Q5 2N7002KQ-13, Q6 2N7002KQ-13, Q7 BC857BQ-13-F, SW3 DIAG KMR221GLFS, U18 BCR420UW6Q-7, U19 AL8861QMP-13

Commit message: Rebuild phase 2 schematic by function
Parts:
- removed Q4: 2N7002KQ-13, Package_TO_SOT_SMD:SOT-23, symbol LandyHeater:2N7002KQ_13_1G_2S_3D
- added C52: 10uF 100V X7R 10%, Capacitor_SMD:C_1210_3225Metric_Pad1.33x2.70mm_HandSolder, symbol LandyHeater:10uF_100V_X7R_10__11_22
- added R75: 47k, Resistor_SMD:R_0603_1608Metric_Pad0.98x0.95mm_HandSolder, symbol LandyHeater:47k_11_22
- added TP35: FRONTLIGHT_PWM, TestPoint:TestPoint_Pad_D1.0mm, symbol LandyHeater:FRONTLIGHT_PWM_11
- added TP36: BUTTON_N, TestPoint:TestPoint_Pad_D1.0mm, symbol LandyHeater:BUTTON_N_11
- added TP37: BUTTON_LED_PWM, TestPoint:TestPoint_Pad_D1.0mm, symbol LandyHeater:BUTTON_LED_PWM_11
- added TP38: DIAG_RUN, TestPoint:TestPoint_Pad_D1.0mm, symbol LandyHeater:DIAG_RUN_11
- D10: value SS14 -> B140Q-13-F; symbol LandyHeater:SS14_1K_2A -> LandyHeater:B140Q_13_F_1K_2A; MPN (none) -> B140Q-13-F; Manufacturer (none) -> Diodes Inc.; Notes AL8861 freewheel diode; KiCad diode pad 1 is K -> Automotive 1-A/40-V Schottky; KiCad diode pad 1 is K
- J4: symbol LandyHeater:1053131305_BUTTON_LED_11_22_33_44_55 -> LandyHeater:1053131305_BUTTON_LED_1BUTTON_N_2GND_3LED_CC_PLUS_4LED_PWM_MINUS_5NC; Notes APEM AV970220000700 cable assembly; pin 5 reserve NC -> APEM AV970220000700 cable assembly; 3m; twist 1/2 and 3/4; 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
- L4: value 47uH >=0.5A -> 47uH 570mA; footprint Inductor_SMD:L_Coilcraft_XAL4020-XXX -> LandyHeater:PROVISIONAL_Murata_LQH3NPZ_JR; symbol LandyHeater:47uH_0_5A_11_22 -> LandyHeater:47uH_570mA_11_22; MPN (none) -> LQH3NPZ470MJR; Manufacturer (none) -> Murata; Notes (none) -> AL8861 33..100uH range; footprint provisional pending offic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
- LED2: Notes (none) -> Raw connector VBUS: indicates actual USB presence, not comm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
- R41: Notes (none) -> Direct hardware default OFF at BCR421 EN
- U18: value BCR420UW6Q-7 -> BCR421UW6Q-7; symbol LandyHeater:BCR420UW6Q_7_1EN_2OUT_3OUT_4GND_5OUT_6REXT -> LandyHeater:BCR421UW6Q_7_1EN_2OUT_3OUT_4GND_5OUT_6REXT; MPN BCR420UW6Q-7 -> BCR421UW6Q-7; Notes (none) -> Preset 10mA; native low-side PWM EN <25kHz
Connections:
- net BUTTON_LED_SINK is gone; now on net LED_PWM_MINUS: U18.2 (OUT), U18.3 (OUT), U18.5 (OUT)
- net LED12_K is gone; now on net VIN_12V_PROTECTED: LED1.1 (K), R46.1
- net LED3V3_K is gone; now on net 3V3_CORE: LED3.1 (K), R48.1
- net LEDHEAT_K is gone; now on net AUTOTERM_5V: LED4.1 (K), R49.1
- net LEDRUN_K is gone; now on net 3V3_CORE: LED5.1 (K), R50.1
- net STATUS1_A is gone; now on net GND: LED6.2 (A), R52.2
- net STATUS2_A is gone; now on net GND: LED7.2 (A), R53.2
- net USB_PROTECTED is gone; now on net USB_VBUS: LED2.2 (A)
- net BUTTON_LED_PWM: now also TP37.1
- net BUTTON_N: now also TP36.1
- net DIAG_GATE: now also R75.2; no longer Q7.3 (C)
- net DIAG_RUN: now also TP38.1
- net FRONTLIGHT_PWM: now also TP35.1
- net GND: now also J4.2 (GND), C52.2; no longer J4.4
- net VIN_SYS: now also C52.1; no longer U18.1 (EN)
- net BUTTON_LED_A renamed LED_CC_PLUS
- net LED_CC_PLUS: now also J4.3 (LED_CC_PLUS); no longer J4.2
- net BUTTON_LED_GATE renamed BUTTON_LED_EN
- net BUTTON_LED_EN: now also U18.1 (EN)
- net BUTTON_LED_K renamed LED_PWM_MINUS
- net LED_PWM_MINUS: now also J4.4 (LED_PWM_MINUS); no longer J4.3
- net BUTTON_WIRE renamed BUTTON_N_EXT
- net DIAG_BASE: no longer names the net of Q7.1 (B), R67.2
- net LEDUSB_K renamed USB_VBUS
- net RUN_ISO: no longer names the net of D15.1 (A), Q6.2 (S)
- new net DIAG_GATE_DRIVE: Q7.3 (C), R75.1
Other:
- note added: "ENERGY-FLOW DIAGNOSTICS — LEDs only while DIAG is pressed"
- note added: "EXTERNAL BUTTON + WHITE RING LED / 3 m"
- note added: "FLOW: J4 BUTTON -> FILTER/ESD -> GPIO1 | GPIO38 -> BCR421 PWM -> J4 RING LED"
- note added: "FLOW: VIN_SYS -> AL8861/L4/D10 -> J8 FRONTLIGHT"
- note added: "FRONTLIGHT 50 mA NOMINAL / <60 mA WORST CASE"
- moved on the sheet: C35, D10, D11, D12, D13, D14, D15, D16, D9, J4, J8, R38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

Commit message: Redraw phase 2 schematic with visible functional wiring
Parts:
- C35: Circuit label (none) -> 10nF
- C52: Circuit label (none) -> CGA6P1X7R2A106K250AC
- D10: Circuit label (none) -> B140Q-13-F
- D11, D12, D13, D14, D15: Circuit label (none) -> BAS116,215
- D16: Circuit label (none) -> PESD24VL1BA,115
- D9: Circuit label (none) -> PESD3V3S1BA
- J4: Circuit label (none) -> BUTTON / RING LED
- J8: Circuit label (none) -> FRONTLIGHT FPC
- L4: Circuit label (none) -> LQH3NPZ470MJR
- LED1, LED2, LED3, LED4, LED5: Circuit label (none) -> LTST-C190KRKT
- LED6, LED7: Circuit label (none) -> LTST-C190KRKT [DNP]
- Q5, Q6: Circuit label (none) -> 2N7002KQ-13
- Q7: Circuit label (none) -> BC857BQ-13-F
- R38: Circuit label (none) -> 1k
- R39: Circuit label (none) -> 10k
- R40: Circuit label (none) -> 100R
- R41, R42, R45, R51, R66: Circuit label (none) -> 100k
- R43: Circuit label (none) -> 2.0R 1% 0.25W
- R44, R65: Circuit label (none) -> 0R
- R46: Circuit label (none) -> 12k
- R47, R49: Circuit label (none) -> 3.3k
- R48, R50: Circuit label (none) -> 1.2k
- R52, R53: Circuit label (none) -> 2.7k DNP [DNP]
- R67, R75: Circuit label (none) -> 47k
- SW3: Circuit label (none) -> KMR221GLFS
- U18: Circuit label (none) -> BCR421UW6Q-7
- U19: Circuit label (none) -> AL8861QMP-13
Connections:
- net 3V3_CORE: no longer LED3.1 (K), LED5.1 (K), R48.1, R50.1
- net AUTOTERM_5V: no longer LED4.1 (K), R49.1
- net GND: no longer LED6.2 (A), LED7.2 (A), R52.2, R53.2
- net USB_VBUS: no longer LED2.1 (K), R47.1
- net VIN_12V_PROTECTED: no longer LED1.1 (K), R46.1
- net BUTTON_LED_EN: no longer names the net of R40.2, R41.1, U18.1 (EN)
- net BUTTON_N_EXT: no longer names the net of D9.1 (IO), J4.1 (BUTTON_N), R38.1
- net DIAG_CATHODE: no longer names the net of D11.3 (K), D12.3 (K), D13.3 (K), D14.3 (K), D15.3 (K), Q5.3 (D)
- net DIAG_GATE: no longer names the net of Q5.1 (G), R45.1, R75.2
- net DIAG_GATE_DRIVE: no longer names the net of Q7.3 (C), R75.1
- net DIAG_N: no longer names the net of R66.2, R67.1, SW3.1 (A), TP21.1
- net FL_ISENSE: no longer names the net of R43.2, R44.1, TP20.1, U19.1 (ISENSE)
- net FL_LED_A: no longer names the net of J8.1, J8.2, R44.2
- net FL_LED_K: no longer names the net of J8.5, J8.6, L4.1
- net FL_LX: no longer names the net of D10.2 (A), L4.2, U19.5 (LX), U19.6 (LX)
- net LED12_ISO: no longer names the net of D11.1 (A), R46.2
- net LED3V3_ISO: no longer names the net of D13.1 (A), R48.2
- net LEDHEAT_ISO: no longer names the net of D14.1 (A), R49.2
- net LEDUSB_ISO: no longer names the net of D12.1 (A), R47.2
- net LED_CC_PLUS: no longer names the net of J4.3 (LED_CC_PLUS), R65.2
- net LED_PWM_MINUS: no longer names the net of D16.1 (IO), J4.4 (LED_PWM_MINUS), U18.2 (OUT), U18.3 (OUT), U18.5 (OUT)
- net RUN_DRAIN: no longer names the net of Q6.3 (D), R50.2
- new net: LED4.1 (K), R49.1
- new net: LED1.1 (K), R46.1
- new net: LED3.1 (K), R48.1
- new net: LED6.2 (A), R52.2
- new net: LED7.2 (A), R53.2
- new net: LED2.1 (K), R47.1
- new net: LED5.1 (K), R50.1
Other:
- note added: "3 m CABLE"
- note added: "50 mA NOMINAL / <60 mA WORST CASE"
- note added: "BOARD ENERGY-FLOW DIAGNOSTICS + OPTIONAL STATUS LEDS"
- note added: "DIAGNOSTIC LEDs ONLY WHILE DIAG IS PRESSED"
- note added: "EXTERNAL BUTTON + PWM WHITE RING LED"
- note added: "FRONTLIGHT CONTROL"
- note removed: "ENERGY-FLOW DIAGNOSTICS — LEDs only while DIAG is pressed"
- note removed: "EXTERNAL BUTTON + WHITE RING LED / 3 m"
- note removed: "FLOW: J4 BUTTON -> FILTER/ESD -> GPIO1 | GPIO38 -> BCR421 PWM -> J4 RING LED"
- note removed: "FLOW: VIN_SYS -> AL8861/L4/D10 -> J8 FRONTLIGHT"
- note removed: "FRONTLIGHT 50 mA NOMINAL / <60 mA WORST CASE"
- moved on the sheet: C35, C52, D10, D11, D12, D13, D14, D15, D16, D9, J4, J8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
