File: kicad/LandyHeater.kicad_sch (KiCad schematic)
At the start: 0 parts

Commit message: Phase 2: draw power sheet (12 V input, USB-C eFuse, 3.3 V buck)
Co-Authored-By: Claude Opus 5.5 <noreply@anthropic.com>
Other:
- added sheet AUTOTERM und 1-Wire (03_AUTOTERM_1Wire.kicad_sch)
- added sheet ESP32 und RTC (02_ESP32_RTC.kicad_sch)
- added sheet Taster und Anzeige (04_Taster_Anzeige.kicad_sch)
- added sheet Versorgung (01_Versorgung.kicad_sch)
Changed lines of the file:
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@@
     (comment 1 "Grundlage: docs/Anforderungsdokument_Neuentwicklung.md v2.0")
+  )
+  (sheet (at 30.0 40.0) (size 50.0 30.0) (fields_autoplaced yes)
+    (stroke (width 0.0006) (type default))
+    (fill (color 0 0 0 0.0000))
+    (property "Sheetname" "Versorgung" (at 32.54 38.73 0)
+      (effects (font (size 1.27 1.27)) (justify left bottom))
+    )
+    (property "Sheetfile" "01_Versorgung.kicad_sch" (at 32.54 71.27 0)
+      (effects (font (size 1.27 1.27)) (justify left top))
+    )
+    (instances
+      (project "LandyHeater"
+        (path "/f79b4c10-b95d-476a-8de2-bd665410a76d" (page "2"))
+      )
+    )
+  )
+  (sheet (at 100.0 40.0) (size 50.0 30.0) (fields_autoplaced yes)
+    (stroke (width 0.0006) (type default))
+    (fill (color 0 0 0 0.0000))
+    (property "Sheetname" "ESP32 und RTC" (at 102.54 38.73 0)
+      (effects (font (size 1.27 1.27)) (justify left bottom))
+    )
+    (property "Sheetfile" "02_ESP32_RTC.kicad_sch" (at 102.54 71.27 0)
+      (effects (font (size 1.27 1.27)) (justify left top))
+    )
+    (instances
+      (project "LandyHeater"
+        (path "/f79b4c10-b95d-476a-8de2-bd665410a76d" (page "3"))
+      )
+    )
+  )
+  (sheet (at 30.0 90.0) (size 50.0 30.0) (fields_autoplaced yes)
+    (stroke (width 0.0006) (type default))
+    (fill (color 0 0 0 0.0000))
+    (property "Sheetname" "AUTOTERM und 1-Wire" (at 32.54 88.73 0)
+      (effects (font (size 1.27 1.27)) (justify left bottom))
+    )
+    (property "Sheetfile" "03_AUTOTERM_1Wire.kicad_sch" (at 32.54 121.27 0)
+      (effects (font (size 1.27 1.27)) (justify left top))
+    )
+    (instances
+      (project "LandyHeater"
+        (path "/f79b4c10-b95d-476a-8de2-bd665410a76d" (page "4"))
+      )
+    )
+  )
+  (sheet (at 100.0 90.0) (size 50.0 30.0) (fields_autoplaced yes)
+    (stroke (width 0.0006) (type default))
+    (fill (color 0 0 0 0.0000))
+    (property "Sheetname" "Taster und Anzeige" (at 102.54 88.73 0)
+      (effects (font (size 1.27 1.27)) (justify left bottom))
+    )
+    (property "Sheetfile" "04_Taster_Anzeige.kicad_sch" (at 102.54 121.27 0)
+      (effects (font (size 1.27 1.27)) (justify left top))
+    )
+    (instances
+      (project "LandyHeater"
+        (path "/f79b4c10-b95d-476a-8de2-bd665410a76d" (page "5"))
+      )
+    )
   )
   (sheet_instances
