File: kicad/02_ESP32_RTC.kicad_sch (KiCad schematic)
At the start: 0 parts

Commit message: Phase 2: draw ESP32, reset/boot and RTC sheet
Co-Authored-By: Claude Opus 5.5 <noreply@anthropic.com>
Parts:
- added BT1: BR1225, LandyHeater:BatteryClip_MYOUNG_MY-1225-01-J, symbol Device:Battery_Cell
- added C12, C13: 22uF, Capacitor_SMD:C_1206_3216Metric, symbol Device:C
- added C14, C16, C19: 100nF, Capacitor_SMD:C_0603_1608Metric, symbol Device:C
- added C15: 1uF, Capacitor_SMD:C_0603_1608Metric, symbol Device:C
- added C17, C18: DNP, Capacitor_SMD:C_0603_1608Metric, symbol Device:C
- added D5, D6: BAS116, Package_TO_SOT_SMD:SOT-23, symbol LandyHeater:BAS116
- added R10, R11: 22R, Resistor_SMD:R_0603_1608Metric, symbol Device:R
- added R12: 499R, Resistor_SMD:R_0603_1608Metric, symbol Device:R
- added R13, R14: 4.7k, Resistor_SMD:R_0603_1608Metric, symbol Device:R
- added R15: 100k, Resistor_SMD:R_0603_1608Metric, symbol Device:R
- added R8, R9: 10k, Resistor_SMD:R_0603_1608Metric, symbol Device:R
- added SW1: RESET, Button_Switch_SMD:SW_Push_1P1T-SH_NO_CK_KMR2xxG, symbol Switch:SW_Push_Shielded
- added SW2: BOOT, Button_Switch_SMD:SW_Push_1P1T-SH_NO_CK_KMR2xxG, symbol Switch:SW_Push_Shielded
- added TP10: U0TXD, TestPoint:TestPoint_Pad_D1.5mm, symbol Connector:TestPoint
- added TP11: U0RXD, TestPoint:TestPoint_Pad_D1.5mm, symbol Connector:TestPoint
- added TP12: I2C_SDA, TestPoint:TestPoint_Pad_D1.5mm, symbol Connector:TestPoint
- added TP13: I2C_SCL, TestPoint:TestPoint_Pad_D1.5mm, symbol Connector:TestPoint
- added TP14: RTC_INT_N, TestPoint:TestPoint_Pad_D1.5mm, symbol Connector:TestPoint
- added TP15: GND, TestPoint:TestPoint_Pad_D1.5mm, symbol Connector:TestPoint
- added TP8: EN, TestPoint:TestPoint_Pad_D1.5mm, symbol Connector:TestPoint
- added TP9: BOOT_N, TestPoint:TestPoint_Pad_D1.5mm, symbol Connector:TestPoint
- added U4: ESP32-S3-WROOM-1U-N16R8, RF_Module:ESP32-S3-WROOM-1U, symbol RF_Module:ESP32-S3-WROOM-1
- added U5: TPS3808G33DBVR, Package_TO_SOT_SMD:SOT-23-6, symbol Power_Supervisor:TPS3808DBV
- added U6: RV-8263-C8, LandyHeater:MicroCrystal_C8_SON-8_2.0x1.2mm, symbol LandyHeater:RV-8263-C8
Connections:
- new net: C19.1, D5.3 (K), D6.3 (K), U6.5 (VDD)
- new net: R9.2, SW2.2, TP9.1, U4.27 (IO0)
- new net: R10.1, U4.13 (USB_D-)
- new net: TP11.1, U4.36 (RXD0)
- new net: R12.2, TP10.1
- new net: C15.1, R8.2, SW1.2, TP8.1, U4.3 (EN), U5.1 (~{RESET})
- new net: BT1.1 (+), D6.1 (A)
- new net: R11.1, U4.14 (USB_D+)
- new net: R12.1, U4.37 (TXD0)
- new net 1WIRE_DQ: U4.4 (IO4)
- new net 3V3_CORE: C12.1, C13.1, C14.1, C16.1, D5.1 (A), R13.1, R14.1, R15.1, R8.1, R9.1, U4.2 (3V3), U5.5 (SENSE), U5.6 (VDD)
- new net AUTOTERM_OE: U4.6 (IO6)
- new net AUTOTERM_RX_3V3: U4.11 (IO18)
- new net AUTOTERM_TX_3V3: U4.10 (IO17)
- new net BUTTON_LED_PWM: U4.7 (IO7)
- new net BUTTON_N: U4.39 (IO1)
- new net DIAG_RUN: U4.18 (IO10)
- new net GND: BT1.2 (-), C12.2, C13.2, C14.2, C15.2, C16.2, C17.2, C18.2, C19.2, SW1.1, SW1.SH (B), SW2.1, SW2.SH (B), TP15.1, U4.1 (GND), U4.40 (GND), U4.41 (GND), U5.2 (GND), U6.2 (CLKOE), U6.4 (VSS)
- new net I2C_SCL: R14.2, TP13.1, U4.17 (IO9), U6.8 (SCL)
- new net I2C_SDA: R13.2, TP12.1, U4.12 (IO8), U6.1 (SDA)
- new net RTC_INT_N: R15.2, TP14.1, U4.38 (IO2), U6.3 (~{INT})
- new net SENSOR_EN: U4.5 (IO5)
- new net STATUS_LED_1: U4.19 (IO11)
- new net STATUS_LED_2: U4.20 (IO12)
- new net USB_DN_C: C17.1, R10.2
- new net USB_DP_C: C18.1, R11.2
- no-connect marks 0 -> 22
Other:
- note added: "3V3-Abblockung, UART0-Testpads, USB-Serien-R"
- note added: "RTC mit Knopfzelle (Dioden-ODER, kein Laden)"
- note added: "Reset (Supervisor 20 ms) und BOOT"
- company: (none) -> Fabian Hartmann
- title: (none) -> ESP32-S3, Reset/BOOT, USB, RTC
