File: kicad/03_AUTOTERM_1Wire.kicad_sch (KiCad schematic)
At the start: 0 parts

Commit message: Phase 2: draw AUTOTERM UART and 1-Wire sheet
Co-Authored-By: Claude Opus 5.5 <noreply@anthropic.com>
Parts:
- added C20, C23, C24: 1uF, Capacitor_SMD:C_0603_1608Metric, symbol Device:C
- added C21, C22: 100nF, Capacitor_SMD:C_0603_1608Metric, symbol Device:C
- added D7: ESD5Z5.0, Diode_SMD:D_SOD-523, symbol Diode:ESD5Zxx
- added D8: PESD5V2S2UT, Package_TO_SOT_SMD:SOT-23, symbol LandyHeater:PESD5V2S2UT
- added D9: PESD3V3S2UT, Package_TO_SOT_SMD:SOT-23, symbol LandyHeater:PESD3V3S2UT
- added J2: AUTOTERM, Connector_Molex:Molex_Nano-Fit_105313-xx04_1x04_P2.50mm_Horizontal, symbol Connector_Generic:Conn_01x04
- added J3: 1-Wire, Connector_Molex:Molex_Nano-Fit_105313-xx03_1x03_P2.50mm_Horizontal, symbol Connector_Generic:Conn_01x03
- added R16, R17: 100R, Resistor_SMD:R_0603_1608Metric, symbol Device:R
- added R18: 1k, Resistor_SMD:R_0603_1608Metric, symbol Device:R
- added R19, R20: 100k, Resistor_SMD:R_0603_1608Metric, symbol Device:R
- added R21: 4.7k, Resistor_SMD:R_0603_1608Metric, symbol Device:R
- added R22: 0R, Resistor_SMD:R_0603_1608Metric, symbol Device:R
- added TP16: AUTOTERM_5V, TestPoint:TestPoint_Pad_D1.5mm, symbol Connector:TestPoint
- added TP17: CTRL_TX, TestPoint:TestPoint_Pad_D1.5mm, symbol Connector:TestPoint
- added TP18: CTRL_RX, TestPoint:TestPoint_Pad_D1.5mm, symbol Connector:TestPoint
- added TP19: TX_3V3, TestPoint:TestPoint_Pad_D1.5mm, symbol Connector:TestPoint
- added TP20: RX_3V3, TestPoint:TestPoint_Pad_D1.5mm, symbol Connector:TestPoint
- added TP21: OE, TestPoint:TestPoint_Pad_D1.5mm, symbol Connector:TestPoint
- added TP22: 1WIRE_DQ_C, TestPoint:TestPoint_Pad_D1.5mm, symbol Connector:TestPoint
- added TP23: 3V3_SENSOR_SW, TestPoint:TestPoint_Pad_D1.5mm, symbol Connector:TestPoint
- added U7: TXU0202QDCURQ1, Package_SO:VSSOP-8_2.3x2mm_P0.5mm, symbol LandyHeater:TXU0202QDCURQ1
- added U8: TPS22945DCKR, Package_TO_SOT_SMD:SOT-353_SC-70-5, symbol LandyHeater:TPS22945DCKR
Connections:
- new net: C24.1, D9.2 (K2), J3.1 (Pin_1), R21.1, TP23.1, U8.1 (VOUT)
- new net: D9.1 (K1), J3.2 (Pin_2), R21.2, R22.2, TP22.1
- new net: D8.2 (K2), J2.4 (Pin_4), R18.2, TP18.1
- new net: R18.1, U7.1 (B2)
- new net: C20.1, C22.1, R16.1, U7.7 (VCCB)
- new net: R17.1, U7.8 (B1Y)
- new net: D8.1 (K1), J2.3 (Pin_3), R17.2, TP17.1
- new net 1WIRE_DQ: R22.1
- new net 3V3_CORE: C21.1, C23.1, U7.3 (VCCA), U8.5 (VIN)
- new net AUTOTERM_5V: D7.1 (K), J2.1 (Pin_1), R16.2, TP16.1
- new net AUTOTERM_OE: R19.1, TP21.1, U7.6 (OE)
- new net AUTOTERM_RX_3V3: TP20.1, U7.4 (A2Y)
- new net AUTOTERM_TX_3V3: TP19.1, U7.5 (A1)
- new net GND: C20.2, C21.2, C22.2, C23.2, C24.2, D7.2 (A), D8.3 (A), D9.3 (A), J2.2 (Pin_2), J3.3 (Pin_3), R19.2, R20.2, U7.2 (GND), U8.2 (GND)
- new net SENSOR_EN: R20.1, U8.4 (ON)
- no-connect marks 0 -> 1
Other:
- note added: "1-Wire: geschaltete, strombegrenzte Sensorversorgung"
- note added: "AUTOTERM-UART: Pegelwandler 3,3 V / 5 V, OE gesperrt ohne Firmware"
- company: (none) -> Fabian Hartmann
- title: (none) -> AUTOTERM-UART und 1-Wire

Commit message: Phase 2: complete schematic with review and netlist check
Draw the 5-sheet hierarchical schematic (power, ESP32/RTC,
AUTOTERM/1-Wire, button/indicators). ERC clean except one justified
footprint-filter warning, exported netlist matches all expected nodes,
SPICE values are numeric and non-simulated parts carry a reason. Add
BOM fields, final design document and phase 2 review.

Co-Authored-By: Claude Opus 5.5 <noreply@anthropic.com>
Parts:
- C20, C21, C22, C23, C24: Spez (none) -> X7R 16 V 0603
- D7: LCSC (none) -> C82044; MPN (none) -> ESD5Z5.0T1G; Manufacturer (none) -> onsemi
- D8: LCSC (none) -> C18441; MPN (none) -> PESD5V2S2UT,215; Manufacturer (none) -> Nexperia
- D9: LCSC (none) -> C84276; MPN (none) -> PESD3V3S2UT,215; Manufacturer (none) -> Nexperia
- J2: LCSC (none) -> C17554326; MPN (none) -> 1053131304; Manufacturer (none) -> Molex
- J3: LCSC (none) -> C17198650; MPN (none) -> 1053131303; Manufacturer (none) -> Molex
- R15: renamed from R16; Spez (none) -> 0603, 1 %, 0,1 W
- R16: renamed from R17; Spez (none) -> 0603, 1 %, 0,1 W
- R17: renamed from R18; Spez (none) -> 0603, 1 %, 0,1 W
- R18: renamed from R19; Spez (none) -> 0603, 1 %, 0,1 W
- R19: renamed from R20; Spez (none) -> 0603, 1 %, 0,1 W
- R20: renamed from R21; Spez (none) -> 0603, 1 %, 0,1 W
- R21: renamed from R22; Spez (none) -> 0603, 1 %, 0,1 W
- TP16, TP17, TP18, TP19, TP20, TP21, TP22, TP23: now left out of the parts list
- U7: LCSC (none) -> C7372013; MPN (none) -> TXU0202QDCURQ1; Manufacturer (none) -> Texas Instruments
- U8: LCSC (none) -> C47507; MPN (none) -> TPS22945DCKR; Manufacturer (none) -> Texas Instruments
Connections:
- net 3V3_SENSOR_SW: now reaches C24.1, D9.2 (K2), J3.1 (Pin_1), R20.1, TP23.1, U8.1 (VOUT)
- net 1WIRE_DQ_C: now reaches D9.1 (K1), J3.2 (Pin_2), R20.2, R21.2, TP22.1
- net CTRL_RX: now reaches D8.2 (K2), J2.4 (Pin_4), R17.2, TP18.1
- net AUTOTERM_5V_F: now reaches C20.1, C22.1, R15.1, U7.7 (VCCB)
- net CTRL_TX: now reaches D8.1 (K1), J2.3 (Pin_3), R16.2, TP17.1
