File: kicad/01_Versorgung.kicad_sch (KiCad schematic)
At the start: 35 parts, among them J1 12V IN, J5 USB4105-GF-A-060, U1 TPD2EUSB30DRTR, U2 TPS259470LRPWR, U3 LMR43620MSC3RPERQ1

Commit message: Phase 2: complete schematic with review and netlist check
Draw the 5-sheet hierarchical schematic (power, ESP32/RTC,
AUTOTERM/1-Wire, button/indicators). ERC clean except one justified
footprint-filter warning, exported netlist matches all expected nodes,
SPICE values are numeric and non-simulated parts carry a reason. Add
BOM fields, final design document and phase 2 review.

Co-Authored-By: Claude Opus 5.5 <noreply@anthropic.com>
Parts:
- C1: value 47uF 35V -> 47uF; Spez (none) -> Alu-Elko SMD 6,3x7,7, 47 uF, 35 V
- C10, C11: Spez (none) -> X7R 10 V 1206
- C2: Spez (none) -> X7R 25 V 0603
- C3, C7: Spez (none) -> X7R 50 V 0603
- C4: value DNP -> 1nF; Spez (none) -> DNP, X7R 50 V 0603; now not fitted
- C5: Spez (none) -> X5R/X7R 10 V 0603
- C6: Spez (none) -> X7R 50 V 1206
- C8, C9: Spez (none) -> X7R 16 V 0603
- D1: LCSC (none) -> C78413; MPN (none) -> SMBJ18CA; Manufacturer (none) -> Brightking
- D2, D4: LCSC (none) -> C2481; MPN (none) -> SS16; Manufacturer (none) -> MDD
- D3: LCSC (none) -> C82044; MPN (none) -> ESD5Z5.0T1G; Manufacturer (none) -> onsemi
- FB1: Spez (none) -> Ferrit 0805, 600 Ohm @ 100 MHz, >= 1 A
- J1: LCSC (none) -> C17345480; MPN (none) -> 1053131302; Manufacturer (none) -> Molex
- J5: LCSC (none) -> C3025063; MPN (none) -> USB4105-GF-A-060; Manufacturer (none) -> GCT
- L1: LCSC (none) -> C3040383; MPN (none) -> FAUL0420-2R2MT; Manufacturer (none) -> CJiang
- R1, R2, R3, R4, R5: Spez (none) -> 0603, 1 %, 0,1 W
- R6: renamed from R7; Spez (none) -> 0603, 1 %, 0,1 W
- TP1, TP2, TP3, TP4, TP5, TP6, TP7: now left out of the parts list
- U1: LCSC (none) -> C97502; MPN (none) -> TPD2EUSB30DRTR; Manufacturer (none) -> Texas Instruments
- U2: LCSC (none) -> C3662793; MPN (none) -> TPS259470LRPWR; Manufacturer (none) -> Texas Instruments
- U3: LCSC (none) -> C3190193; MPN (none) -> LMR43620MSC3RPERQ1; Manufacturer (none) -> Texas Instruments
Connections:
- net USB_VBUS: now reaches C2.1, D3.1 (K), J5.A4 (VBUS), J5.A9 (VBUS), J5.B4 (VBUS), J5.B9 (VBUS), R3.1, TP5.1, U2.5 (IN)
- net BATT_12V_IN: now reaches D1.2 (A2), D2.2 (A), J1.1 (Pin_1), TP1.1
- net CC1: now reaches J5.A5 (CC1), R1.1
- net SW_BUCK: now reaches C9.1, L1.1, U3.5 (SW)
- net CC2: now reaches J5.B5 (CC2), R2.1

Commit message: Add C26 100 nF at 12V_PROT ahead of the ferrite (E-01)
Forms a pi filter with FB1 and C1 and limits the reverse voltage across D2
in ISO 7637-2 pulse 3a from 60.3 V to 38.8 V (SPICE, sim/v01_transienten.py).
Placed between D2 and FB1; ERC, netlist check and DRC clean.

Co-Authored-By: Claude Opus 5.5 <noreply@anthropic.com>
Parts:
- added C26: 100nF, Capacitor_SMD:C_0603_1608Metric, symbol Device:C
Connections:
- net 12V_PROT: now also C26.1
- net GND: now also C26.2
Changed lines of the file:
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@@
+		)
+	)
+	(symbol
+		(lib_id "Device:C")
+		(at 69.85 62.23 0)
+		(unit 1)
+		(body_style 1)
+		(exclude_from_sim no)
+		(in_bom yes)
+		(on_board yes)
+		(in_pos_files yes)
+		(dnp no)
+		(property "Reference" "C26"
+			(at 73.25 60.96 0)
+			(show_name no)
+			(do_not_autoplace no)
+			(effects
+				(font
+					(size 1.27 1.27)
+				)
+			)
+		)
+		(property "Value" "100nF"
+			(at 74.9 63.5 0)
+			(show_name no)
+			(do_not_autoplace no)
+			(effects
+				(font
+					(size 1.27 1.27)
+				)
+			)
+		)
+		(property "Footprint" "Capacitor_SMD:C_0603_1608Metric"
+			(at 70.81 58.42 0)
+			(hide yes)
+			(show_name no)
+			(do_not_autoplace no)
+			(effects
+				(font
+					(size 1.27 1.27)
+				)
+			)
+		)
+		(property "Datasheet" ""
+			(at 69.85 62.23 0)
+			(hide yes)
+			(show_name no)
+			(do_not_autoplace no)
+			(effects
+				(font
+					(size 1.27 1.27)
+				)
+			)
+		)
+		(property "Description" "Unpolarized capacitor"
+			(at 69.85 62.23 0)
+			(hide yes)
+			(show_name no)
+			(do_not_autoplace no)
+			(effects
+				(font
+					(size 1.27 1.27)
+				)
+			)
+		)
+		(property "Spez" "X7R 50 V 0603"
+			(at 69.85 62.23 0)
+			(hide yes)
+			(show_name no)
+			(do_not_autoplace no)
+			(effects
+				(font
+					(size 1.27 1.27)
+				)
+			)
+		)
+		(pin "1"
+		)
+		(pin "2"
+		)
+		(instances
+			(project "LandyHeater"
+				(path "/f79b4c10-b95d-476a-8de2-bd665410a76d/c39d3920-4fd8-4364-ab23-17d6e9c351a7"
+					(reference "C26")
+					(unit 1)
+				)
+			)
+		)
+	)
+	(symbol
+		(lib_id "power:GND")
+		(at 69.85 66.04 0)
+		(unit 1)
+		(body_style 1)
+		(exclude_from_sim no)
+		(in_bom yes)
+		(on_board yes)
+		(in_pos_files yes)
+		(dnp no)
+		(property "Reference" "#PWR081"
+			(at 69.85 66.04 0)
+			(hide yes)
+			(show_name no)
+			(do_not_autoplace no)
+			(effects
+				(font
+					(size 1.27 1.27)
+				)
+			)
+		)
+		(property "Value" "GND"
+			(at 69.85 71.12 0)
+			(show_name no)
+			(do_not_autoplace no)
+			(effects
+				(font
+					(size 1.27 1.27)
+				)
+			)
+		)
+		(property "Footprint" ""
+			(at 69.85 66.04 0)
+			(hide yes)
+			(show_name no)
+			(do_not_autoplace no)
+			(effects
+				(font
+					(size 1.27 1.27)
+				)
+			)
+		)
+		(property "Datasheet" ""
+			(at 69.85 66.04 0)
+			(hide yes)
+			(show_name no)
+			(do_not_autoplace no)
+			(effects
+				(font
+					(size 1.27 1.27)
+				)
+			)
+		)
+		(property "Description" "Power symbol creates a global label with name \"GND\" , ground"
+			(at 69.85 66.04 0)
+			(hide yes)
+			(show_name no)
+			(do_not_autoplace no)
+			(effects
+				(font
+					(size 1.27 1.27)
+				)
+			)
+		)
+		(pin "1"
+		)
+		(instances
+			(project "LandyHeater"
+				(path "/f79b4c10-b95d-476a-8de2-bd665410a76d/c39d3920-4fd8-4364-ab23-17d6e9c351a7"
+					(reference "#PWR081")
+					(unit 1)
+				)
+			)
 		)
 	)
