File: kicad/04_Taster_Anzeige.kicad_sch (KiCad schematic)
At the start: 0 parts

Commit message: Phase 2: complete schematic with review and netlist check
Draw the 5-sheet hierarchical schematic (power, ESP32/RTC,
AUTOTERM/1-Wire, button/indicators). ERC clean except one justified
footprint-filter warning, exported netlist matches all expected nodes,
SPICE values are numeric and non-simulated parts carry a reason. Add
BOM fields, final design document and phase 2 review.

Co-Authored-By: Claude Opus 5.5 <noreply@anthropic.com>
Parts:
- added C25: 10nF, Capacitor_SMD:C_0603_1608Metric, symbol Device:C
- added D10: PESD3V3S2UT, Package_TO_SOT_SMD:SOT-23, symbol LandyHeater:PESD3V3S2UT
- added D11, D12, D13, D14, D19, D20, D21: rot, LED_SMD:LED_0603_1608Metric, symbol Device:LED
- added D15, D16, D17, D18: BAS116, Package_TO_SOT_SMD:SOT-23, symbol LandyHeater:BAS116
- added F1: 50mA, Fuse:Fuse_0805_2012Metric, symbol Device:Polyfuse
- added J4: Taster/LED, Connector_Molex:Molex_Nano-Fit_105313-xx05_1x05_P2.50mm_Horizontal, symbol Connector_Generic:Conn_01x05
- added Q1: 2N7002K, Package_TO_SOT_SMD:SOT-23, symbol Transistor_FET:2N7002K
- added R22, R28, R32, R33: 1k, Resistor_SMD:R_0603_1608Metric, symbol Device:R
- added R23: 10k, Resistor_SMD:R_0603_1608Metric, symbol Device:R
- added R24: 100R, Resistor_SMD:R_0603_1608Metric, symbol Device:R
- added R25, R31, R34, R35: 100k, Resistor_SMD:R_0603_1608Metric, symbol Device:R
- added R26: 12k, Resistor_SMD:R_0603_1608Metric, symbol Device:R
- added R27, R29: 3.3k, Resistor_SMD:R_0603_1608Metric, symbol Device:R
- added R30: 1.8k, Resistor_SMD:R_0603_1608Metric, symbol Device:R
- added SW3: DIAG, Button_Switch_SMD:SW_Push_1P1T-SH_NO_CK_KMR2xxG, symbol Switch:SW_Push_Shielded
- added TP24: DIAG, TestPoint:TestPoint_Pad_D1.5mm, symbol Connector:TestPoint
- added TP25: GND, TestPoint:TestPoint_Pad_D1.5mm, symbol Connector:TestPoint
- added TP26: BUTTON_N, TestPoint:TestPoint_Pad_D1.5mm, symbol Connector:TestPoint
- added TP27: BUTTON_LED_PWM, TestPoint:TestPoint_Pad_D1.5mm, symbol Connector:TestPoint
- added TP28: DIAG_RUN, TestPoint:TestPoint_Pad_D1.5mm, symbol Connector:TestPoint
- added U9: BCR421UW6Q-7, Package_TO_SOT_SMD:SOT-23-6, symbol LandyHeater:BCR421UW6Q-7
Connections:
- new net: D11.1 (K), D15.1 (A)
- new net: D11.2 (A), R26.2
- new net: D14.1 (K), D18.1 (A)
- new net: D14.2 (A), R29.2
- new net: D13.1 (K), D17.1 (A)
- new net: D13.2 (A), R28.2
- new net: R24.2, R25.1, U9.1 (EN)
- new net: D12.1 (K), D16.1 (A)
- new net: D12.2 (A), R27.2
- new net: D19.1 (K), Q1.3 (D)
- new net: D19.2 (A), R30.2
- new net: D20.2 (A), R32.2
- new net: D21.2 (A), R33.2
- new net 12V_PROT: R26.1
- new net 3V3_CORE: R23.1, R28.1, R30.1
- new net AUTOTERM_5V: R29.1
- new net BUTTON_LED_PWM: R24.1, TP27.1
- new net BUTTON_N: C25.1, R22.1, R23.2, TP26.1
- new net BUTTON_N_C: D10.1 (K1), J4.1 (Pin_1), R22.2
- new net DIAG_K: D15.3 (K), D16.3 (K), D17.3 (K), D18.3 (K), Q1.2 (S), SW3.2, TP24.1
- new net DIAG_RUN: Q1.1 (G), R31.1, TP28.1
- new net GND: C25.2, D10.3 (A), D20.1 (K), D21.1 (K), J4.2 (Pin_2), R25.2, R31.2, R34.2, R35.2, SW3.1, SW3.SH (B), TP25.1, U9.4 (GND)
- new net LED_CC_PLUS: F1.2, J4.3 (Pin_3)
- new net LED_PWM_MINUS: J4.4 (Pin_4), U9.2 (OUT), U9.3 (OUT), U9.5 (OUT)
- new net STATUS_LED_1: R32.1, R34.1
- new net STATUS_LED_2: R33.1, R35.1
- new net VBUS_PROT: R27.1
- new net VIN_SYS: F1.1
- no-connect marks 0 -> 3
Other:
- note added: "Energiefluss-Diagnose (nur bei gedruecktem DIAG)"
- note added: "Externer Taster (3 m) und Ring-LED 10 mA (PWM)"
- note added: "Status-LEDs"
- company: (none) -> Fabian Hartmann
- title: (none) -> Taster, Ring-LED, Diagnose- und Status-LEDs

Commit message: F1 = BORN SMD0805-005/60N (LCSC C22366098); routing approved
- F1 uses project symbol LandyHeater:Polyfuse_0805 (footprint filter
  matches Fuse_0805); ERC 0/0, DRC incl. schematic parity 0
- board F1 fields synced (Spez, MPN, Manufacturer, LCSC)
- report: footprint/connector review, 3D model gaps, approval

Co-Authored-By: Claude Opus 5.5 <noreply@anthropic.com>
Parts:
- F1: symbol Device:Polyfuse -> LandyHeater:Polyfuse_0805; LCSC (none) -> C22366098; MPN (none) -> SMD0805-005/60N; Manufacturer (none) -> BORN; Spez PTC 0805, I_hold ca. 50 mA, I_trip ca. 150 mA, >= 16 V -> PTC 0805, I_hold 50 mA, I_trip 150 mA, 60 V (BORN SMD0805-0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
Changed lines of the file:
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@@
 	)
 	(symbol
-		(lib_id "Device:Polyfuse")
+		(lib_id "LandyHeater:Polyfuse_0805")
 		(at 182.88 76.2 90)
 		(unit 1)
@@
 			)
 		)
-		(property "Spez" "PTC 0805, I_hold ca. 50 mA, I_trip ca. 150 mA, >= 16 V"
+		(property "Spez" "PTC 0805, I_hold 50 mA, I_trip 150 mA, 60 V (BORN SMD0805-005/60N)"
 			(at 182.88 76.2 0)
 			(hide yes)
+			(show_name no)
+			(do_not_autoplace no)
+			(effects
+				(font
+					(size 1.27 1.27)
+				)
+			)
+		)
+		(property "MPN" "SMD0805-005/60N"
+			(at 182.88 76.2 0)
+			(hide yes)
+			(show_name no)
+			(do_not_autoplace no)
+			(effects
+				(font
+					(size 1.27 1.27)
+				)
+			)
+		)
+		(property "Manufacturer" "BORN"
+			(at 182.88 76.2 0)
+			(hide yes)
+			(show_name no)
+			(do_not_autoplace no)
+			(effects
+				(font
+					(size 1.27 1.27)
+				)
+			)
+		)
+		(property "LCSC" "C22366098"
+			(at 182.88 76.2 0)
+			(hide yes)
